File: Hardware/2024/mod-badge-inercia/mod-badge-inercia.kicad_sch (KiCad schematic)
At the start: 91 parts, among them J1 USB_C_Receptacle_USB2.0, J101 Conn_01x02_Shielded, J102 Conn_01x02_Shielded, J103 Conn_02x03_Odd_Even, J2 Micro_SD_Card_Det1, J3 Conn_01x03_MountingPin, J4 Conn_01x02_Shielded, J6 Conn_01x04, J7 Conn_02x06_Odd_Even, Q1 DMG3415U, SW2 SW_MEC_5E, SW3 SW_MEC_5E, SW4 SW_MEC_5E, SW5 SW_MEC_5E, SW6 SW_MEC_5E, SW7 SW_Push_DPDT, U1 RP2040, U2 USBLC6-2P6, U4 W25Q32JVSS, U5 MAX98357AETE_T, U6 TPS63802DLAR, Y1 12MHZ

Commit message: minor changes and fixes
Parts:
- R1: footprint Resistor_SMD:R_0402_1005Metric -> Resistor_SMD:R_0603_1608Metric; LCSC C5126239 -> C2684557
- RV1: now left out of the parts list
Changed lines of the file:
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@@
 			)
 		)
-		(property "Footprint" "Resistor_SMD:R_0402_1005Metric"
+		(property "Footprint" "Resistor_SMD:R_0603_1608Metric"
 			(at 212.852 50.8 90)
 			(effects
@@
 			)
 		)
-		(property "LCSC" "C5126239"
+		(property "LCSC" "C2684557"
 			(at 214.63 50.8 0)
 			(effects
@@
 		(unit 1)
 		(exclude_from_sim no)
-		(in_bom yes)
+		(in_bom no)
 		(on_board yes)
 		(dnp no)

Commit message: Minor changes and bom consolidation
Parts:
- added D3: D_Schottky, Diode_SMD:D_SOD-123F, symbol Device:D_Schottky
- added R25, R4: 100, Resistor_SMD:R_0402_1005Metric, symbol Device:R
- Q1: symbol Device:Q_PMOS_SGD -> Device:Q_PMOS_GSD
- R9: footprint Resistor_SMD:R_0603_1608Metric -> Resistor_SMD:R_0402_1005Metric; LCSC C22548 -> C11702
Connections:
- net +BATT: now also D3.2 (A)
- net MCU_SWCLK: now also R4.1; no longer U1.24 (SWCLK)
- net MCU_SWD: now also R25.1; no longer U1.25 (SWD)
- net VBUS: now also Q1.1 (G); no longer Q1.2 (G)
- net at D1.1 (K), R3.1: now also Q1.2 (S), D3.1 (K); no longer Q1.1 (S)
- new net: R4.2, U1.24 (SWCLK)
- new net: R25.2, U1.25 (SWD)
Other:
- moved on the sheet: C22, C23, D2, L101, R1, R103, R104, R2, R20, R24, R3, U6

Commit message: updated sao connector. minor changes
Parts:
- removed J103: Conn_02x03_Odd_Even, Connector_PinSocket_2.54mm:PinSocket_2x03_P2.54mm_Vertical, symbol Connector_Generic:Conn_02x03_Odd_Even
- added TP5: TestPoint, TestPoint:TestPoint_Pad_D1.0mm, symbol Connector:TestPoint
- added X1: Badgelife_sao_connector_v169bis, mod:Badgelife-SAOv169-BADGE-2x3, symbol mod:Badgelife_sao_connector_v169bis
Connections:
- net +3V3: now also X1.1 (VCC)
- net GND: now also X1.2 (GND)
- net GP9: now also TP5.1
- net SAO_GPIO1: now also X1.5 (GPIO1)
- net SAO_GPIO2: now also X1.6 (GPIO2)
- net SAO_SCL: now also X1.4 (SCL)
- net SAO_SDA: now also X1.3 (SDA)
Other:
- note added: "just an extra gpio"

Commit message: minor fixes, sent final 2024 badges to production
Parts:
- R106, R107: LCSC C5126239 -> C37825
Changed lines of the file:
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@@
 			)
 		)
-		(property "LCSC" "C5126239"
+		(property "LCSC" "C37825"
 			(at 86.36 43.18 0)
 			(effects
@@
 			)
 		)
-		(property "LCSC" "C5126239"
+		(property "LCSC" "C37825"
 			(at 102.87 43.18 0)
 			(effects
